File: FOCDriver/Power.kicad_sch (KiCad schematic)
At the start: 58 parts, among them J12 Screw_Terminal_01x02, J5 Screw_Terminal_01x02, Q2 SIR422DP-T1-GE3, U13 LM22676MR-5, U14 Si4435DDY, U17 ZXCT1109, U6 AMS1117-3.3

Commit message: Update
Parts:
- added C90: 100n, Footprints:Nice_0603C, symbol Device:C
- added D8, D9: APT2012SYCK, LED_SMD:LED_0805_2012Metric, symbol Device:LED
- added R80: DNP, Footprints:Nice_0402DNP, symbol Device:R
- added R81, R82: 1k, Footprints:Nice_0402R, symbol Device:R
- C43: footprint Capacitor_SMD:CP_Elec_10x10 -> Capacitor_SMD:CP_Elec_8x10.5; MPN (none) -> EEEFT1V331AP
- C68, C69, C83: footprint Capacitor_SMD:CP_Elec_10x10 -> Capacitor_SMD:CP_Elec_10x10.5; MPN (none) -> EEV FK1V331P
- D1: value 10V zener -> BZX384-B10,115; MPN BZX384 -> BZX384-B10,115
- D7: value LED -> APT2012SYCK; MPN (none) -> APT2012SYCK
- F1: value 30R300U / 30R500U -> 30R500U
- L1: value L_Ferrite -> BLM18AG471SN1D
- R62: value 100 -> 100R
- U13: MPN (none) -> LM22672MRX-5.0/NOPB
Connections:
- net +5V: now also R81.1
- net GND: now also C90.2, D8.1 (K), D9.1 (K), R80.1
- net VDD: now also R82.1
- net at U14.5 (D), U14.6 (D), U14.7 (D)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: now also J5.1 (Pin_1); no longer D1.1 (K), F1.1
- net at U14.1 (S), U14.2 (S), U14.3 (S): now also D1.1 (K), F1.1; no longer J5.1 (Pin_1)
- net at U13.2 (SS): now also C90.1
- net at U13.3 (RT): now also R80.2
- new net: D8.2 (A), R81.2
- new net: D9.2 (A), R82.2
Other:
- note added: "(incase BLDC drvs regen power)"
- note added: "(useful for scope etc.)"
- note added: "10V Zener BZX384-B10"
- note added: "12V -> 5V 1A Buck Converter"
- note added: "20m nominal R (0.5W loss at 5A)"
- note added: "35V"
- note added: "3x EEE HA1V331P: 250mA ripple 3x EEV FK1V331P: 850mA ripple"
- note added: "5V -> 3.3V LDO"
- note added: "Bulk Decoupling"
- note added: "Current Sense: 408uA @ 100mV diff 3.0V / 408uA = 7.5k => 2x 15kR parallel"
- note added: "Current Shunt"
- note added: "DO214AC (SMA)"
- note added: "Ground Points"
- note added: "Input Fuse 3A-5A hold current"
- note added: "LM22672MRX-5.0/NOPB"
- note added: "PI filter"
- note added: "Power Input"
- note added: "Power Monitor"
- note added: "Resistive Clamp"
- note added: "Reverse Polarity Protection"
- note added: "Si4435: 20mOhm @ -10Vgs => Ploss=I^2 R = 0.5W at 5A"
- note added: "Voltage Sense: 10k/1k = 1/11 scaling 24V => 2182mV"
- note added: "may need tuning 74279223560 ferrite: 1612 package Z=56R max, 10A rating 4mOhms (100mW loss)"
- note removed: "12V-3.3V Rja=135C/W Ta=50C, Tj=100C => 0.37W (42.5mA)"
- note removed: "3.0V / 408uA = 7.5k (2x 15kR parallel?)"
- note removed: "408uA @ 100mV diff"
- moved on the sheet: C18, C30, C43, C64, C65, C66, C67, C68, C69, C70, C77, C78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
